Commit message: Fix URDF mesh orientations and robot_description launch param
Add rpy origins to align servo holder, arm, and camera meshes, adjust
joint origins, and wrap robot_description Command in ParameterValue so
it is published as a string.

Co-Authored-By: Claude Opus 4.8 (1M context) <noreply@anthropic.com>

File: ros2/pibob_description/urdf/pibob.urdf.xacro (robot description, xacro)
@@ -9,5 +9,4 @@
   -->
   <xacro:property name="mesh_pkg" value="package://pibob_description/meshes"/>
-  <xacro:property name="pi"       value="3.14159265359"/>
   <!-- ============ Materials ============ -->
   <material name="white"><color rgba="0.95 0.95 0.95 1"/></material>
@@ -24,9 +23,9 @@
     <parent link="base_link"/>
     <child  link="shoulder_beam"/>
-    <origin xyz="0 0 0.05" rpy="0 0 0"/>
+    <origin xyz="0 0 0.30" rpy="0 0 0"/>
   </joint>
   <link name="shoulder_beam">
     <visual>
-      <origin xyz="0 0 0" rpy="0 0 0"/>
+      <origin xyz="0 0 0" rpy="1.5708 0 0"/>
       <geometry><mesh filename="${mesh_pkg}/Shoulder-Beam.stl" scale="0.001 0.001 0.001"/></geometry>
       <material name="grey"/>
@@ -37,5 +36,5 @@
     <parent link="shoulder_beam"/>
     <child  link="head_pan_link"/>
-    <origin xyz="0 0 0.06" rpy="0 0 0"/>
+    <origin xyz="0 0 0.10" rpy="0 0 0"/>
     <axis xyz="0 0 1"/>
     <!-- safe range CH2: 0..180 deg => -pi/2..+pi/2 about home (90 deg) -->
@@ -44,4 +43,5 @@
   <link name="head_pan_link">
     <visual>
+      <origin xyz="0 0 0" rpy="0 -1.5708 0"/>
       <geometry><mesh filename="${mesh_pkg}/Head-BottomServoHolder.stl" scale="0.001 0.001 0.001"/></geometry>
       <material name="white"/>
@@ -58,4 +58,5 @@
   <link name="head_tilt_link">
     <visual>
+      <origin xyz="0 0 0" rpy="0 -1.5708 0"/>
       <geometry><mesh filename="${mesh_pkg}/Head-MiddleServoHolder.stl" scale="0.001 0.001 0.001"/></geometry>
       <material name="white"/>
@@ -69,4 +70,5 @@
   <link name="camera_link">
     <visual>
+      <origin xyz="0 0 0" rpy="1.5708 0 1.5708"/>
       <geometry><mesh filename="${mesh_pkg}/Head-CameraHolder.stl" scale="0.001 0.001 0.001"/></geometry>
       <material name="grey"/>
@@ -86,5 +88,5 @@
       <parent link="shoulder_beam"/>
       <child  link="${side}_shoulder_rot_link"/>
-      <origin xyz="0 ${0.09*reflect} 0.0" rpy="0 0 0"/>
+      <origin xyz="0 ${0.09*reflect} 0.09" rpy="0 0 0"/>
       <axis xyz="0 1 0"/>
       <!-- CH7/CH11 safe 70..150 -->
@@ -93,4 +95,5 @@
     <link name="${side}_shoulder_rot_link">
       <visual>
+        <origin xyz="0 0 0" rpy="-1.5708 0 0"/>
         <geometry><mesh filename="${mesh_pkg}/${holder_mesh}" scale="0.001 0.001 0.001"/></geometry>
         <material name="white"/>
@@ -107,4 +110,5 @@
     <link name="${side}_shoulder_lift_link">
       <visual>
+        <origin xyz="0 0 0" rpy="-1.5708 0 0"/>
         <geometry><mesh filename="${mesh_pkg}/${bracket_mesh}" scale="0.001 0.001 0.001"/></geometry>
         <material name="grey"/>
@@ -121,4 +125,5 @@
     <link name="${side}_upper_arm_link">
       <visual>
+        <origin xyz="0 0 0" rpy="0 1.5708 0"/>
         <geometry><mesh filename="${mesh_pkg}/Arm-Bicep.stl" scale="0.001 0.001 0.001"/></geometry>
         <material name="white"/>
@@ -135,10 +140,10 @@
     <link name="${side}_forearm_link">
       <visual>
-        <origin xyz="0 0 0" rpy="0 0 0"/>
+        <origin xyz="0 0 0" rpy="-1.5708 0 0"/>
         <geometry><mesh filename="${mesh_pkg}/Arm-Elbow.stl" scale="0.001 0.001 0.001"/></geometry>
         <material name="grey"/>
       </visual>
       <visual>
-        <origin xyz="0 0 -0.04" rpy="0 0 0"/>
+        <origin xyz="0 0 -0.04" rpy="-1.5708 0 0"/>
         <geometry><mesh filename="${mesh_pkg}/Arm-Forearm.stl" scale="0.001 0.001 0.001"/></geometry>
         <material name="white"/>

Commit message: Docker: live-edit hot-reload for the URDF + in-progress model tweaks
Dev workflow so the URDF can be tuned without rebuilds:
- entrypoint: a file-watcher (WATCH=1) that re-runs xacro and bounces the
  launch whenever pibob.urdf.xacro changes; RViz redraws in ~12s. Nodes are
  hard-killed by name between reloads so windows don't pile up; xacro errors
  are logged and the last good model kept.
- dev.sh: one-command launcher that mounts the urdf/ dir and sets WATCH=1.
- README: live-edit section.
This beats native Mac URDF viewers because the container already has ROS +
xacro + the package, so package:// meshes and the xacro macro resolve.

Model tweaks so far (still being tuned via live-edit): biceps rotated 90deg,
shoulder brackets long-ways, arms offset outward (0.10), head left at original
height.

Co-Authored-By: Claude Opus 4.8 (1M context) <noreply@anthropic.com>

File: ros2/pibob_description/urdf/pibob.urdf.xacro (robot description, xacro)
@@ -110,5 +110,7 @@
     <link name="${side}_shoulder_lift_link">
       <visual>
-        <origin xyz="0 0 0" rpy="-1.5708 0 0"/>
+        <!-- bracket spans outward (long 115mm side along the span) so it bridges
+             from the shoulder to the arm sitting further out -->
+        <origin xyz="0 0 0" rpy="0 0 0"/>
         <geometry><mesh filename="${mesh_pkg}/${bracket_mesh}" scale="0.001 0.001 0.001"/></geometry>
         <material name="grey"/>
@@ -118,5 +120,6 @@
       <parent link="${side}_shoulder_lift_link"/>
       <child  link="${side}_upper_arm_link"/>
-      <origin xyz="0 0 -0.04" rpy="0 0 0"/>
+      <!-- arm sits further out along the bracket (outward in Y), then drops -->
+      <origin xyz="0 ${0.10*reflect} -0.04" rpy="0 0 0"/>
       <axis xyz="0 0 1"/>
       <!-- CH5/CH9 safe 70..110 -->
@@ -125,5 +128,6 @@
     <link name="${side}_upper_arm_link">
       <visual>
-        <origin xyz="0 0 0" rpy="0 1.5708 0"/>
+        <!-- bicep rotated 90 deg -->
+        <origin xyz="0 0 0" rpy="0 1.5708 1.5708"/>
         <geometry><mesh filename="${mesh_pkg}/Arm-Bicep.stl" scale="0.001 0.001 0.001"/></geometry>
         <material name="white"/>

Commit message: urdf: fix arm mesh chain to match README assembly order
Top-ServoHolder now FIXED to the beam (was mis-placed on shoulder_rot); bracket and
L/R ServoHolder were swapped. Correct chain: beam -> Top(fixed) -> [CH7]bracket ->
[CH6]L/R holder -> [CH5]bicep -> [CH4]elbow/forearm. Verified renders cleanly (RobotModel Ok).

Co-Authored-By: Claude Opus 4.8 (1M context) <noreply@anthropic.com>

File: ros2/pibob_description/urdf/pibob.urdf.xacro (robot description, xacro)
@@ -36,5 +36,5 @@
     <parent link="shoulder_beam"/>
     <child  link="head_pan_link"/>
-    <origin xyz="0 0 0.10" rpy="0 0 0"/>
+    <origin xyz="0 0 0.045" rpy="0 0 0"/>
     <axis xyz="0 0 1"/>
     <!-- safe range CH2: 0..180 deg => -pi/2..+pi/2 about home (90 deg) -->
@@ -85,17 +85,30 @@
   -->
   <xacro:macro name="arm" params="side reflect bracket_mesh holder_mesh">
+    <!-- Top servo holder: FIXED into the Shoulder-Beam end (houses the CH7/CH11 servo) -->
+    <joint name="${side}_shoulder_top_joint" type="fixed">
+      <parent link="shoulder_beam"/>
+      <child  link="${side}_shoulder_top_link"/>
+      <origin xyz="0 ${0.09*reflect} 0.09" rpy="0 0 0"/>
+    </joint>
+    <link name="${side}_shoulder_top_link">
+      <visual>
+        <origin xyz="0 0 0" rpy="-1.5708 0 0"/>
+        <geometry><mesh filename="${mesh_pkg}/Shoulder-Top-ServoHolder.stl" scale="0.001 0.001 0.001"/></geometry>
+        <material name="white"/>
+      </visual>
+    </link>
+    <!-- CH7/CH11 shoulder_rot: top holder rotates the BRACKET (arm up/down front) -->
     <joint name="${side}_shoulder_rot_joint" type="revolute">
-      <parent link="shoulder_beam"/>
+      <parent link="${side}_shoulder_top_link"/>
       <child  link="${side}_shoulder_rot_link"/>
-      <origin xyz="0 ${0.09*reflect} 0.09" rpy="0 0 0"/>
-      <axis xyz="0 1 0"/>
-      <!-- CH7/CH11 safe 70..150 -->
+      <origin xyz="0 0 0" rpy="0 0 0"/>
+      <axis xyz="0 ${reflect} 0"/>
       <limit lower="-0.3491" upper="1.0472" effort="1.0" velocity="3.14"/>
     </joint>
     <link name="${side}_shoulder_rot_link">
       <visual>
-        <origin xyz="0 0 0" rpy="-1.5708 0 0"/>
-        <geometry><mesh filename="${mesh_pkg}/${holder_mesh}" scale="0.001 0.001 0.001"/></geometry>
-        <material name="white"/>
+        <origin xyz="0 0 0" rpy="0 0 0"/>
+        <geometry><mesh filename="${mesh_pkg}/${bracket_mesh}" scale="0.001 0.001 0.001"/></geometry>
+        <material name="grey"/>
       </visual>
     </link>
@@ -104,5 +117,5 @@
       <child  link="${side}_shoulder_lift_link"/>
       <origin xyz="0 0 -0.03" rpy="0 0 0"/>
-      <axis xyz="1 0 0"/>
+      <axis xyz="${reflect} 0 0"/>   <!-- mirror per side so both arms wing out symmetrically -->
       <!-- CH6/CH10 safe 70..110 -->
       <limit lower="-0.3491" upper="0.3491" effort="1.0" velocity="3.14"/>
@@ -110,9 +123,7 @@
     <link name="${side}_shoulder_lift_link">
       <visual>
-        <!-- bracket spans outward (long 115mm side along the span) so it bridges
-             from the shoulder to the arm sitting further out -->
         <origin xyz="0 0 0" rpy="0 0 0"/>
-        <geometry><mesh filename="${mesh_pkg}/${bracket_mesh}" scale="0.001 0.001 0.001"/></geometry>
-        <material name="grey"/>
+        <geometry><mesh filename="${mesh_pkg}/${holder_mesh}" scale="0.001 0.001 0.001"/></geometry>
+        <material name="white"/>
       </visual>
     </link>

Commit message: urdf: per-part show flags (show_top/bracket/holder/bicep/forearm) to seat arm meshes one at a time
Co-Authored-By: Claude Opus 4.8 (1M context) <noreply@anthropic.com>

File: ros2/pibob_description/urdf/pibob.urdf.xacro (robot description, xacro)
@@ -9,4 +9,10 @@
   -->
   <xacro:property name="mesh_pkg" value="package://pibob_description/meshes"/>
+  <!-- ===== arm-part debug toggles: show one mesh at a time while seating it ===== -->
+  <xacro:property name="show_top"     value="true"/>
+  <xacro:property name="show_bracket" value="false"/>
+  <xacro:property name="show_holder"  value="false"/>
+  <xacro:property name="show_bicep"   value="false"/>
+  <xacro:property name="show_forearm" value="false"/>
   <!-- ============ Materials ============ -->
   <material name="white"><color rgba="0.95 0.95 0.95 1"/></material>
@@ -92,4 +98,5 @@
     </joint>
     <link name="${side}_shoulder_top_link">
+      <xacro:if value="${show_top}">
       <visual>
         <origin xyz="0 0 0" rpy="-1.5708 0 0"/>
@@ -97,4 +104,5 @@
         <material name="white"/>
       </visual>
+      </xacro:if>
     </link>
     <!-- CH7/CH11 shoulder_rot: top holder rotates the BRACKET (arm up/down front) -->
@@ -107,4 +115,5 @@
     </joint>
     <link name="${side}_shoulder_rot_link">
+      <xacro:if value="${show_bracket}">
       <visual>
         <origin xyz="0 0 0" rpy="0 0 0"/>
@@ -112,4 +121,5 @@
         <material name="grey"/>
       </visual>
+      </xacro:if>
     </link>
     <joint name="${side}_shoulder_lift_joint" type="revolute">
@@ -122,4 +132,5 @@
     </joint>
     <link name="${side}_shoulder_lift_link">
+      <xacro:if value="${show_holder}">
       <visual>
         <origin xyz="0 0 0" rpy="0 0 0"/>
@@ -127,4 +138,5 @@
         <material name="white"/>
       </visual>
+      </xacro:if>
     </link>
     <joint name="${side}_arm_rot_joint" type="revolute">
@@ -138,4 +150,5 @@
     </joint>
     <link name="${side}_upper_arm_link">
+      <xacro:if value="${show_bicep}">
       <visual>
         <!-- bicep rotated 90 deg -->
@@ -144,4 +157,5 @@
         <material name="white"/>
       </visual>
+      </xacro:if>
     </link>
     <joint name="${side}_bicep_joint" type="revolute">
@@ -154,4 +168,5 @@
     </joint>
     <link name="${side}_forearm_link">
+      <xacro:if value="${show_forearm}">
       <visual>
         <origin xyz="0 0 0" rpy="-1.5708 0 0"/>
@@ -164,4 +179,5 @@
         <material name="white"/>
       </visual>
+      </xacro:if>
     </link>
   </xacro:macro>

Commit message: urdf: seat arm meshes (top/bracket/holder/bicep) with per-side mirroring
- Correct chain per README: beam -> Top-ServoHolder(fixed) -> bracket -> L/R holder -> bicep.
- Per-side reflect for Y offsets + 180/90 yaw inverts where meshes mirror.
- Gimbal-lock at +/-90 pitch on the holder: baked 180 into Shoulder-Left-ServoHolder.stl
  (orig kept locally as .orig); bicep is a single mesh so left mirrored via 180 rotation.
- Debug show_* toggles to seat one part at a time; forearm still to do.

Co-Authored-By: Claude Opus 4.8 (1M context) <noreply@anthropic.com>

File: ros2/pibob_description/urdf/pibob.urdf.xacro (robot description, xacro)
@@ -11,7 +11,7 @@
   <!-- ===== arm-part debug toggles: show one mesh at a time while seating it ===== -->
   <xacro:property name="show_top"     value="true"/>
-  <xacro:property name="show_bracket" value="false"/>
-  <xacro:property name="show_holder"  value="false"/>
-  <xacro:property name="show_bicep"   value="false"/>
+  <xacro:property name="show_bracket" value="true"/>
+  <xacro:property name="show_holder"  value="true"/>
+  <xacro:property name="show_bicep"   value="true"/>
   <xacro:property name="show_forearm" value="false"/>
   <!-- ============ Materials ============ -->
@@ -72,9 +72,9 @@
     <parent link="head_tilt_link"/>
     <child  link="camera_link"/>
-    <origin xyz="0.04 0 0.02" rpy="0 0 0"/>
+    <origin xyz="0.00 0 0.03" rpy="0 0 0"/>
   </joint>
   <link name="camera_link">
     <visual>
-      <origin xyz="0 0 0" rpy="1.5708 0 1.5708"/>
+      <origin xyz="0 0 0" rpy="1.5708 1.5708 1.5708"/>
       <geometry><mesh filename="${mesh_pkg}/Head-CameraHolder.stl" scale="0.001 0.001 0.001"/></geometry>
       <material name="grey"/>
@@ -95,10 +95,11 @@
       <parent link="shoulder_beam"/>
       <child  link="${side}_shoulder_top_link"/>
-      <origin xyz="0 ${0.09*reflect} 0.09" rpy="0 0 0"/>
+      <origin xyz="0 ${0.085*reflect} 0.065" rpy="0 0 0"/>
     </joint>
     <link name="${side}_shoulder_top_link">
       <xacro:if value="${show_top}">
       <visual>
-        <origin xyz="0 0 0" rpy="-1.5708 0 0"/>
+        <!-- roll 180 = small end down; per-side yaw flips the pin to mirror the two holders -->
+        <origin xyz="0 0 0" rpy="3.14159 0 ${(1+reflect)/2*3.14159}"/>
         <geometry><mesh filename="${mesh_pkg}/Shoulder-Top-ServoHolder.stl" scale="0.001 0.001 0.001"/></geometry>
         <material name="white"/>
@@ -117,5 +118,6 @@
       <xacro:if value="${show_bracket}">
       <visual>
-        <origin xyz="0 0 0" rpy="0 0 0"/>
+        <!-- per-side yaw: invert the our-left (reflect=-1) bracket 180 to mirror -->
+        <origin xyz="0.0 ${0.02*reflect} 0.018" rpy="0 0 ${(1-reflect)/2*3.14159}"/>
         <geometry><mesh filename="${mesh_pkg}/${bracket_mesh}" scale="0.001 0.001 0.001"/></geometry>
         <material name="grey"/>
@@ -134,5 +136,5 @@
       <xacro:if value="${show_holder}">
       <visual>
-        <origin xyz="0 0 0" rpy="0 0 0"/>
+        <origin xyz="0 ${0.097*reflect} 0.035" rpy="0 -1.5708 3.14159"/>
         <geometry><mesh filename="${mesh_pkg}/${holder_mesh}" scale="0.001 0.001 0.001"/></geometry>
         <material name="white"/>
@@ -144,5 +146,5 @@
       <child  link="${side}_upper_arm_link"/>
       <!-- arm sits further out along the bracket (outward in Y), then drops -->
-      <origin xyz="0 ${0.10*reflect} -0.04" rpy="0 0 0"/>
+      <origin xyz="0.004 ${0.14*reflect} 0.005" rpy="0 0 0"/>
       <axis xyz="0 0 1"/>
       <!-- CH5/CH9 safe 70..110 -->
@@ -152,6 +154,6 @@
       <xacro:if value="${show_bicep}">
       <visual>
-        <!-- bicep rotated 90 deg -->
-        <origin xyz="0 0 0" rpy="0 1.5708 1.5708"/>
+        <!-- bicep: right (reflect=+1) = pi; left gets -180 to mirror -->
+        <origin xyz="0 0 0" rpy="0 1.5708 ${3.14159 - (1-reflect)/2*3.14159}"/>
         <geometry><mesh filename="${mesh_pkg}/Arm-Bicep.stl" scale="0.001 0.001 0.001"/></geometry>
         <material name="white"/>

Commit message: urdf: split elbow onto bicep link; forearm swings with joint; mirror + axis fixes
- Arm-Elbow now fixed on upper_arm_link (houses CH4 servo, stays put); Arm-Forearm on
  forearm_link swings with the elbow joint.
- Elbow (bicep_joint) axis flipped so the elbow bends forward.
- Forearm/elbow Y offsets use *reflect; per-side yaw mirrors the single-mesh parts.
- show_forearm (elbow) / show_forearm_mesh (forearm) toggles for seating each.

Co-Authored-By: Claude Opus 4.8 (1M context) <noreply@anthropic.com>

File: ros2/pibob_description/urdf/pibob.urdf.xacro (robot description, xacro)
@@ -14,5 +14,6 @@
   <xacro:property name="show_holder"  value="true"/>
   <xacro:property name="show_bicep"   value="true"/>
-  <xacro:property name="show_forearm" value="false"/>
+  <xacro:property name="show_forearm" value="true"/>   <!-- the elbow piece -->
+  <xacro:property name="show_forearm_mesh" value="true"/>  <!-- the swinging forearm -->
   <!-- ============ Materials ============ -->
   <material name="white"><color rgba="0.95 0.95 0.95 1"/></material>
@@ -160,4 +161,12 @@
       </visual>
       </xacro:if>
+      <!-- elbow: FIXED to the bicep (houses CH4 servo) — does NOT move with the joint. Tune xyz to seat it. -->
+      <xacro:if value="${show_forearm}">
+      <visual>
+        <origin xyz="0 ${-0.014*reflect} -0.076" rpy="-1.5708 0 ${1.5708*reflect}"/>
+        <geometry><mesh filename="${mesh_pkg}/Arm-Elbow.stl" scale="0.001 0.001 0.001"/></geometry>
+        <material name="grey"/>
+      </visual>
+      </xacro:if>
     </link>
     <joint name="${side}_bicep_joint" type="revolute">
@@ -165,17 +174,13 @@
       <child  link="${side}_forearm_link"/>
       <origin xyz="0 0 -0.08" rpy="0 0 0"/>
-      <axis xyz="0 1 0"/>
+      <axis xyz="0 -1 0"/>   <!-- flipped: elbow bends forward, not back -->
       <!-- CH4/CH8 safe 90..180 => 0..+pi/2 (cannot go below straight) -->
       <limit lower="0.0" upper="1.5708" effort="1.0" velocity="3.14"/>
     </joint>
     <link name="${side}_forearm_link">
-      <xacro:if value="${show_forearm}">
+      <xacro:if value="${show_forearm_mesh}">
+      <!-- only the FOREARM swings with the elbow joint; left gets 90 yaw to mirror -->
       <visual>
-        <origin xyz="0 0 0" rpy="-1.5708 0 0"/>
-        <geometry><mesh filename="${mesh_pkg}/Arm-Elbow.stl" scale="0.001 0.001 0.001"/></geometry>
-        <material name="grey"/>
-      </visual>
-      <visual>
-        <origin xyz="0 0 -0.04" rpy="-1.5708 0 0"/>
+        <origin xyz="0 ${-0.02*reflect} -0.0425" rpy="-1.5708 0 ${1.5708*reflect}"/>
         <geometry><mesh filename="${mesh_pkg}/Arm-Forearm.stl" scale="0.001 0.001 0.001"/></geometry>
         <material name="white"/>

Commit message: urdf: shoulder-lift pivot knobs (lift_pivot_in/up) — move pivot to the connector without moving the arm
Joint origin moves to the rotation point; holder visual + arm_rot origin auto-compensate
so the arm stays put. Negative lift_pivot_in = outward toward the connector.

Co-Authored-By: Claude Opus 4.8 (1M context) <noreply@anthropic.com>

File: ros2/pibob_description/urdf/pibob.urdf.xacro (robot description, xacro)
@@ -9,4 +9,9 @@
   -->
   <xacro:property name="mesh_pkg" value="package://pibob_description/meshes"/>
+  <!-- move the shoulder-lift PIVOT without moving the arm (holder + arm auto-compensated).
+       lift_pivot_in: POSITIVE = toward body centre, NEGATIVE = OUTWARD toward the connector/red dot.
+       lift_pivot_up: upward to the connector. -->
+  <xacro:property name="lift_pivot_in" value="-0.06"/>
+  <xacro:property name="lift_pivot_up" value="0.05"/>
   <!-- ===== arm-part debug toggles: show one mesh at a time while seating it ===== -->
   <xacro:property name="show_top"     value="true"/>
@@ -129,5 +134,6 @@
       <parent link="${side}_shoulder_rot_link"/>
       <child  link="${side}_shoulder_lift_link"/>
-      <origin xyz="0 0 -0.03" rpy="0 0 0"/>
+      <!-- this origin IS the lift pivot: move Y toward the head to pivot from the inner edge -->
+      <origin xyz="0 ${-lift_pivot_in*reflect} ${-0.03+lift_pivot_up}" rpy="0 0 0"/>
       <axis xyz="${reflect} 0 0"/>   <!-- mirror per side so both arms wing out symmetrically -->
       <!-- CH6/CH10 safe 70..110 -->
@@ -137,5 +143,5 @@
       <xacro:if value="${show_holder}">
       <visual>
-        <origin xyz="0 ${0.097*reflect} 0.035" rpy="0 -1.5708 3.14159"/>
+        <origin xyz="0 ${(0.097+lift_pivot_in)*reflect} ${0.035-lift_pivot_up}" rpy="0 -1.5708 3.14159"/>
         <geometry><mesh filename="${mesh_pkg}/${holder_mesh}" scale="0.001 0.001 0.001"/></geometry>
         <material name="white"/>
@@ -147,5 +153,5 @@
       <child  link="${side}_upper_arm_link"/>
       <!-- arm sits further out along the bracket (outward in Y), then drops -->
-      <origin xyz="0.004 ${0.14*reflect} 0.005" rpy="0 0 0"/>
+      <origin xyz="0.004 ${(0.14+lift_pivot_in)*reflect} ${0.005-lift_pivot_up}" rpy="0 0 0"/>
       <axis xyz="0 0 1"/>
       <!-- CH5/CH9 safe 70..110 -->
