Commit message: head: seat the head on modelled 9 g servos, derived from the holder STLs
- New meshes/Servo-9g.stl (scripts/make_servo_stl.py): SG90/MG90S-class 9 g servo,
  origin on the output shaft at the body top face. Size from the holder pockets
  (23.0 x 12.2 / 23.0 x 12.1 mm) and the bottom holder's coaxial pin (shaft 5.85 mm
  from the pocket end).
- xacro: reusable servo_9g visual macro; pan + tilt servos, and elbow servos (elbow
  holder is the same part as the head bottom holder; shaft on the bicep axis to
  0.1 mm). No arm joint moved.
- Head re-seated from mating features: bottom holder (pocket up, pin in the beam's
  head hole) on new fixed head_base_link; pan joint on the pan shaft at its top face
  (z 62.2 mm above beam centre); middle holder rides the pan horn via its hub hole
  and carries the tilt servo (head_pan_link); tilt joint on the tilt shaft at its top
  face; camera holder's arm hub hole on the tilt shaft (head_tilt_link); camera_link
  at the board centre.
- Checks: head pivots 0.000 mm off their servo shaft, all head contact gaps 0.0 mm,
  RViz TF 0.0000 mm/0.0000 deg all poses, head close-up IoU 0.997-0.998.
- Verification: servo/contact checks, head close-up views, fixed RViz panel crop for
  close-ups, head_closeup.png sheet.

Co-Authored-By: Claude Opus 5.5 <noreply@anthropic.com>
Claude-Session: https://claude.ai/code/session_01Wgu7BJrMw6Ry2NoXo3DYtX

File: ros2/pibob_description/urdf/pibob.urdf.xacro (robot description, xacro)
@@ -25,4 +25,15 @@
   <material name="white"><color rgba="0.95 0.95 0.95 1"/></material>
   <material name="grey"><color rgba="0.4 0.4 0.4 1"/></material>
+  <material name="servo_grey"><color rgba="0.2 0.2 0.2 1"/></material>
+  <!-- 9 g micro servo (SG90 / MG90S class) visual. Mesh frame: origin on the output
+       shaft at the body's top (horn) face, +z out along the shaft, +x along the body
+       from the shaft end. Generated by scripts/make_servo_stl.py. -->
+  <xacro:macro name="servo_9g" params="xyz rpy">
+    <visual>
+      <origin xyz="${xyz}" rpy="${rpy}"/>
+      <geometry><mesh filename="${mesh_pkg}/Servo-9g.stl" scale="0.001 0.001 0.001"/></geometry>
+      <material name="servo_grey"/>
+    </visual>
+  </xacro:macro>
   <!-- ============ Base + torso ============ -->
   <link name="base_link">
@@ -46,32 +57,65 @@
   </link>
   <!-- ============ Head ============ -->
+  <!--
+    Seated from the holder STL geometry (see fusion/README.md "Head"), not by eye:
+      Head-BottomServoHolder = 9 g servo pocket (23.0 x 12.2, 17.25 deep) open at its +y
+        face, with a dia-4.7 pivot pin on the opposite face coaxial with the servo shaft.
+        Pocket UP: the pan servo stands in it, tabs on the holder top, shaft vertical; the
+        holder sits on the beam top with the pin in the beam's 20 x 20 head hole.
+      Head-MiddleServoHolder = horn groove + dia-7 hub hole in its floor (rides the pan
+        horn) and a second 9 g pocket (23.0 x 12.1, 18 deep) open to the robot's left
+        (+y) for the tilt servo.
+      Head-CameraHolder = camera U-frame whose side arm has a dia-7 hub hole + horn
+        groove on its outer face: it rides the tilt servo's horn.
+    Each revolute joint origin is on its servo's output-shaft axis at the servo's top
+    (horn / mounting) face.
+  -->
+  <joint name="beam_to_head_base" type="fixed">
+    <parent link="shoulder_beam"/>
+    <child  link="head_base_link"/>
+    <origin xyz="0 0 0.0355" rpy="0 0 0"/>   <!-- beam top face, on the head hole centre -->
+  </joint>
+  <!-- fixed to the beam: the bottom holder + the pan servo standing in it -->
+  <link name="head_base_link">
+    <visual>
+      <origin xyz="0 -0.0041 0.0075" rpy="${pi/2} 0 ${pi/2}"/>
+      <geometry><mesh filename="${mesh_pkg}/Head-BottomServoHolder.stl" scale="0.001 0.001 0.001"/></geometry>
+      <material name="white"/>
+    </visual>
+    <xacro:servo_9g xyz="0 0 0.0267" rpy="0 0 ${pi/2}"/>    <!-- pan servo (CH2) -->
+  </link>
   <joint name="head_pan_joint" type="revolute">
     <parent link="shoulder_beam"/>
     <child  link="head_pan_link"/>
-    <origin xyz="0 0 0.045" rpy="0 0 0"/>
+    <!-- pan servo shaft axis, at its top face: beam top 35.5 + holder/servo stack 26.7 mm -->
+    <origin xyz="0 0 0.0622" rpy="0 0 0"/>
     <axis xyz="0 0 1"/>
     <!-- safe range CH2: 0..180 deg => -pi/2..+pi/2 about home (90 deg) -->
     <limit lower="-1.5708" upper="1.5708" effort="1.0" velocity="3.14"/>
   </joint>
+  <!-- turns with pan: the middle holder (on the pan horn) + the tilt servo inside it -->
   <link name="head_pan_link">
     <visual>
-      <origin xyz="0 0 0" rpy="0 -1.5708 0"/>
-      <geometry><mesh filename="${mesh_pkg}/Head-BottomServoHolder.stl" scale="0.001 0.001 0.001"/></geometry>
+      <origin xyz="0 0.0005 0.010" rpy="0 0 0"/>
+      <geometry><mesh filename="${mesh_pkg}/Head-MiddleServoHolder.stl" scale="0.001 0.001 0.001"/></geometry>
       <material name="white"/>
     </visual>
+    <xacro:servo_9g xyz="-0.00315 0.0172 0.01105" rpy="${-pi/2} 0 0"/>    <!-- tilt servo (CH3) -->
   </link>
   <joint name="head_tilt_joint" type="revolute">
     <parent link="head_pan_link"/>
     <child  link="head_tilt_link"/>
-    <origin xyz="0 0 0.03" rpy="0 0 0"/>
+    <!-- tilt servo shaft axis, at its top face (where the camera arm sits on the horn) -->
+    <origin xyz="-0.00315 0.0172 0.01105" rpy="0 0 0"/>
     <axis xyz="0 1 0"/>
     <!-- safe range CH3: 50..140 deg => -40..+50 deg around home -->
     <limit lower="-0.6981" upper="0.8727" effort="1.0" velocity="3.14"/>
   </joint>
+  <!-- turns with tilt: the camera holder, its arm's hub hole on the tilt shaft -->
   <link name="head_tilt_link">
     <visual>
-      <origin xyz="0 0 0" rpy="0 -1.5708 0"/>
-      <geometry><mesh filename="${mesh_pkg}/Head-MiddleServoHolder.stl" scale="0.001 0.001 0.001"/></geometry>
-      <material name="white"/>
+      <origin xyz="0 -0.01775 0.02867" rpy="0 ${pi/2} 0"/>
+      <geometry><mesh filename="${mesh_pkg}/Head-CameraHolder.stl" scale="0.001 0.001 0.001"/></geometry>
+      <material name="grey"/>
     </visual>
   </link>
@@ -79,13 +123,8 @@
     <parent link="head_tilt_link"/>
     <child  link="camera_link"/>
-    <origin xyz="0.00 0 0.03" rpy="0 0 0"/>
-  </joint>
-  <link name="camera_link">
-    <visual>
-      <origin xyz="0 0 0" rpy="1.5708 1.5708 1.5708"/>
-      <geometry><mesh filename="${mesh_pkg}/Head-CameraHolder.stl" scale="0.001 0.001 0.001"/></geometry>
-      <material name="grey"/>
-    </visual>
-  </link>
+    <!-- centre of the camera board in the holder's U-frame -->
+    <origin xyz="-0.00625 -0.0195 0.04467" rpy="0 0 0"/>
+  </joint>
+  <link name="camera_link"/>
   <!-- ============ Arm macro ============ -->
   <!--
@@ -175,4 +214,6 @@
         <material name="grey"/>
       </visual>
+      <!-- elbow servo (CH4/CH8) in the elbow holder's pocket; its shaft is the bicep axis -->
+      <xacro:servo_9g xyz="0 ${-0.0332*reflect} -0.0801" rpy="${pi/2} ${pi/2} ${(1-reflect)/2*pi}"/>
       </xacro:if>
     </link>

Commit message: arms: put every arm joint origin on its physical pin (parts unmoved)
- pin_check.py fits the cylindrical features in the STLs: DS3218 holders carry a
  dia-5.8 pin coaxial with the servo shaft; driven U-brackets have a dia-21 horn
  seat + dia-9 hub hole and a dia-6 pin hole; 9 g elbow has a dia-4.7 pin.
- shoulder_rot / shoulder_lift / arm_rot / bicep origins moved onto the pin root
  (moved 14.3 / 19.5 / 57.8 / 6.5 mm); every visual and child-joint origin
  re-expressed so zero-pose geometry is identical (max vertex displacement 0.0 mm).
  Axis angle vs pin 0.000 deg everywhere; lift_pivot_in/up knobs removed.
- Reports URDF part-seating errors the pins expose (not applied - would move parts):
  bracket 5.6 mm below the top-holder pin, bracket holes 9.5 mm off the holder's
  lift pin, bicep 0.8-0.9 mm, forearm 1.1 mm.
- Per-joint close-ups in fusion/verify/pins/; RViz comparisons re-run (TF 0.0000 mm).

Co-Authored-By: Claude Opus 5.5 <noreply@anthropic.com>
Claude-Session: https://claude.ai/code/session_01Wgu7BJrMw6Ry2NoXo3DYtX

File: ros2/pibob_description/urdf/pibob.urdf.xacro (robot description, xacro)
@@ -9,9 +9,11 @@
   -->
   <xacro:property name="mesh_pkg" value="package://pibob_description/meshes"/>
-  <!-- move the shoulder-lift PIVOT without moving the arm (holder + arm auto-compensated).
-       lift_pivot_in: POSITIVE = toward body centre, NEGATIVE = OUTWARD toward the connector/red dot.
-       lift_pivot_up: upward to the connector. -->
-  <xacro:property name="lift_pivot_in" value="-0.06"/>
-  <xacro:property name="lift_pivot_up" value="0.05"/>
+  <!-- Arm joint pivots are ON the servo shaft axes, located from the mesh geometry: each
+       DS3218 holder carries a dia-5.8 pin coaxial with its servo shaft, and each driven
+       U-bracket has a dia-21 horn seat + dia-9 hub hole on one arm and a dia-6 pin hole on
+       the other. Each joint origin is the centre of that pin where it leaves its holder
+       (elbow: the dia-4.7 pin of the 9 g elbow holder). Every visual / child-joint origin
+       was re-expressed so the parts did NOT move (see fusion/README.md "Arm pivots").
+       The old lift_pivot_in / lift_pivot_up knobs are gone: the pin fixes the pivot. -->
   <!-- ===== arm-part debug toggles: flip a part to false to hide it while seating another.
        All default true, so the full arm renders normally. ===== -->
@@ -157,5 +159,6 @@
       <parent link="${side}_shoulder_top_link"/>
       <child  link="${side}_shoulder_rot_link"/>
-      <origin xyz="0 0 0" rpy="0 0 0"/>
+      <!-- on the top holder's dia-5.8 pin (= CH7/CH11 shaft axis), at the pin root -->
+      <origin xyz="0 ${0.01345*reflect} 0.0049" rpy="0 0 0"/>
       <axis xyz="0 ${reflect} 0"/>
       <limit lower="-0.3491" upper="1.0472" effort="1.0" velocity="3.14"/>
@@ -165,5 +168,5 @@
       <visual>
         <!-- per-side yaw: invert the our-left (reflect=-1) bracket 180 to mirror -->
-        <origin xyz="0.0 ${0.02*reflect} 0.018" rpy="0 0 ${(1-reflect)/2*3.14159}"/>
+        <origin xyz="0.0 ${0.00655*reflect} 0.0131" rpy="0 0 ${(1-reflect)/2*3.14159}"/>
         <geometry><mesh filename="${mesh_pkg}/${bracket_mesh}" scale="0.001 0.001 0.001"/></geometry>
         <material name="grey"/>
@@ -174,6 +177,6 @@
       <parent link="${side}_shoulder_rot_link"/>
       <child  link="${side}_shoulder_lift_link"/>
-      <!-- this origin IS the lift pivot: move Y toward the head to pivot from the inner edge -->
-      <origin xyz="0 ${-lift_pivot_in*reflect} ${-0.03+lift_pivot_up}" rpy="0 0 0"/>
+      <!-- on the shoulder servo holder's dia-5.8 X pin (= CH6/CH10 shaft axis), at the pin root -->
+      <origin xyz="-0.01345 ${0.05605*reflect} 0.00465" rpy="0 0 0"/>
       <axis xyz="${reflect} 0 0"/>   <!-- mirror per side so both arms wing out symmetrically -->
       <!-- CH6/CH10 safe 70..110 -->
@@ -183,5 +186,5 @@
       <xacro:if value="${show_holder}">
       <visual>
-        <origin xyz="0 ${(0.097+lift_pivot_in)*reflect} ${0.035-lift_pivot_up}" rpy="0 -1.5708 3.14159"/>
+        <origin xyz="0.01345 ${0.0275*reflect} -0.00455" rpy="0 -1.5708 3.14159"/>
         <geometry><mesh filename="${mesh_pkg}/${holder_mesh}" scale="0.001 0.001 0.001"/></geometry>
         <material name="white"/>
@@ -192,6 +195,6 @@
       <parent link="${side}_shoulder_lift_link"/>
       <child  link="${side}_upper_arm_link"/>
-      <!-- arm sits further out along the bracket (outward in Y), then drops -->
-      <origin xyz="0.004 ${(0.14+lift_pivot_in)*reflect} ${0.005-lift_pivot_up}" rpy="0 0 0"/>
+      <!-- on the shoulder servo holder's dia-5.8 Z pin (= CH5/CH9 shaft axis), at the pin root -->
+      <origin xyz="0.017 ${0.0511*reflect} 0.0199" rpy="0 0 0"/>
       <axis xyz="0 0 1"/>
       <!-- CH5/CH9: opened to ~+/-51deg (was +/-20 "safe 70..110") — widen/narrow as needed -->
@@ -202,18 +205,18 @@
       <visual>
         <!-- bicep: right (reflect=+1) = pi; left gets -180 to mirror -->
-        <origin xyz="0 0 0" rpy="0 1.5708 ${3.14159 - (1-reflect)/2*3.14159}"/>
+        <origin xyz="0.00045 ${0.0194*reflect} -0.05445" rpy="0 1.5708 ${3.14159 - (1-reflect)/2*3.14159}"/>
         <geometry><mesh filename="${mesh_pkg}/Arm-Bicep.stl" scale="0.001 0.001 0.001"/></geometry>
         <material name="white"/>
       </visual>
       </xacro:if>
-      <!-- elbow: FIXED to the bicep (houses CH4 servo) — does NOT move with the joint. Tune xyz to seat it. -->
+      <!-- elbow: FIXED to the bicep (houses CH4 servo) — does NOT move with the joint. -->
       <xacro:if value="${show_forearm}">
       <visual>
-        <origin xyz="0 ${-0.014*reflect} -0.076" rpy="-1.5708 0 ${1.5708*reflect}"/>
+        <origin xyz="0.00045 ${0.0054*reflect} -0.13045" rpy="-1.5708 0 ${1.5708*reflect}"/>
         <geometry><mesh filename="${mesh_pkg}/Arm-Elbow.stl" scale="0.001 0.001 0.001"/></geometry>
         <material name="grey"/>
       </visual>
       <!-- elbow servo (CH4/CH8) in the elbow holder's pocket; its shaft is the bicep axis -->
-      <xacro:servo_9g xyz="0 ${-0.0332*reflect} -0.0801" rpy="${pi/2} ${pi/2} ${(1-reflect)/2*pi}"/>
+      <xacro:servo_9g xyz="0.00045 ${-0.0138*reflect} -0.13455" rpy="${pi/2} ${pi/2} ${(1-reflect)/2*pi}"/>
       </xacro:if>
     </link>
@@ -221,5 +224,6 @@
       <parent link="${side}_upper_arm_link"/>
       <child  link="${side}_forearm_link"/>
-      <origin xyz="0 0 -0.08" rpy="0 0 0"/>
+      <!-- on the elbow holder's dia-4.7 pin (= CH4/CH8 9 g servo shaft axis), at the pin root -->
+      <origin xyz="0.00045 ${0.0129*reflect} -0.13455" rpy="0 0 0"/>
       <axis xyz="0 -1 0"/>   <!-- flipped: elbow bends forward, not back -->
       <!-- CH4/CH8 safe 90..180 => 0..+pi/2 (cannot go below straight) -->
@@ -230,5 +234,5 @@
       <!-- only the FOREARM swings with the elbow joint; per-side +/-90 yaw mirrors the single mesh -->
       <visual>
-        <origin xyz="0 ${-0.02*reflect} -0.0425" rpy="-1.5708 0 ${1.5708*reflect}"/>
+        <origin xyz="0 ${-0.0135*reflect} -0.0424" rpy="-1.5708 0 ${1.5708*reflect}"/>
         <geometry><mesh filename="${mesh_pkg}/Arm-Forearm.stl" scale="0.001 0.001 0.001"/></geometry>
         <material name="white"/>

Commit message: head: peg-down base, chosen by an exhaustive orientation search; servo gains its gear boss
- verify/head_search.py: every axis-aligned orientation of each head part (24^5 =
  24,576 heads), servos pushed into their pockets, scored for voxel interpenetration
  and the photo cues (peg in beam hole, pan vertical, tilt horizontal, camera up/fwd).
- Servo-9g.stl now has the SG90/MG90S gear boss (dia 11.8 x 4 mm); origin = horn face.
  Without it every peg-down/pan-up head collided (middle holder 3.3 mm into the base).
- Head: Head-BottomServoHolder peg DOWN in the beam's head hole, pocket forward, pan
  servo upright in it (pushed in to its boss, shaft 5.9 mm proud) -> pan axis at
  (15.9, 0, 370.35); middle holder on the pan spline; tilt at (12.75, 21.2, 381.4).
  0 interpenetration > 0.2 mm at zero / pan +-90 / tilt limits; pivots 0.000 mm off
  the splines; hub-hole drift <= 0.001 mm.
- Elbow servo origins moved 4 mm along the shaft so the case stays put (boss now
  overlaps the forearm arm 0.7 mm; fixed by the pending arm re-seat).
- Arm re-seat NOT applied (blocked: approval was relayed, not direct).
- head_vs_photos.png side-by-side; RViz TF 0.0000 mm, head close-up IoU 0.997+.

Co-Authored-By: Claude Opus 5.5 <noreply@anthropic.com>
Claude-Session: https://claude.ai/code/session_01Wgu7BJrMw6Ry2NoXo3DYtX

File: ros2/pibob_description/urdf/pibob.urdf.xacro (robot description, xacro)
@@ -62,7 +62,11 @@
     Seated from the holder STL geometry (see fusion/README.md "Head"), not by eye:
       Head-BottomServoHolder = 9 g servo pocket (23.0 x 12.2, 17.25 deep) open at its +y
-        face, with a dia-4.7 pivot pin on the opposite face coaxial with the servo shaft.
-        Pocket UP: the pan servo stands in it, tabs on the holder top, shaft vertical; the
-        holder sits on the beam top with the pin in the beam's 20 x 20 head hole.
+        face, a 14.5 mm square peg on its -x end, a dia-4.7 pin on its -y face.
+        PEG DOWN into the beam's 20 x 20 head hole (as in Images/), pocket facing FORWARD.
+        The pan servo stands upright in the pocket (23 mm tall = the servo's case height),
+        shaft up; it is pushed in until its gear boss meets the holder's top plate, so its
+        shaft end sits 5.9 mm proud of the holder face - the pan axis is 15.9 mm in front
+        of the beam hole. Chosen by fusion/verify/head_search.py (every axis-aligned
+        orientation of every head part, scored for interpenetration + the photo cues).
       Head-MiddleServoHolder = horn groove + dia-7 hub hole in its floor (rides the pan
         horn) and a second 9 g pocket (23.0 x 12.1, 18 deep) open to the robot's left
@@ -70,6 +74,5 @@
       Head-CameraHolder = camera U-frame whose side arm has a dia-7 hub hole + horn
         groove on its outer face: it rides the tilt servo's horn.
-    Each revolute joint origin is on its servo's output-shaft axis at the servo's top
-    (horn / mounting) face.
+    Each revolute joint origin is on its servo's output-shaft axis at the horn face.
   -->
   <joint name="beam_to_head_base" type="fixed">
@@ -81,15 +84,15 @@
   <link name="head_base_link">
     <visual>
-      <origin xyz="0 -0.0041 0.0075" rpy="${pi/2} 0 ${pi/2}"/>
+      <origin xyz="-0.0025 0 0.00975" rpy="0 ${-pi/2} ${-pi/2}"/>   <!-- peg down, pocket forward -->
       <geometry><mesh filename="${mesh_pkg}/Head-BottomServoHolder.stl" scale="0.001 0.001 0.001"/></geometry>
       <material name="white"/>
     </visual>
-    <xacro:servo_9g xyz="0 0 0.0267" rpy="0 0 ${pi/2}"/>    <!-- pan servo (CH2) -->
+    <xacro:servo_9g xyz="0.0159 0 0.03485" rpy="0 0 ${pi}"/>    <!-- pan servo (CH2), shaft up -->
   </link>
   <joint name="head_pan_joint" type="revolute">
     <parent link="shoulder_beam"/>
     <child  link="head_pan_link"/>
-    <!-- pan servo shaft axis, at its top face: beam top 35.5 + holder/servo stack 26.7 mm -->
-    <origin xyz="0 0 0.0622" rpy="0 0 0"/>
+    <!-- pan servo shaft axis, at its horn face (top of the gear boss) -->
+    <origin xyz="0.0159 0 0.07035" rpy="0 0 0"/>
     <axis xyz="0 0 1"/>
     <!-- safe range CH2: 0..180 deg => -pi/2..+pi/2 about home (90 deg) -->
@@ -103,11 +106,11 @@
       <material name="white"/>
     </visual>
-    <xacro:servo_9g xyz="-0.00315 0.0172 0.01105" rpy="${-pi/2} 0 0"/>    <!-- tilt servo (CH3) -->
+    <xacro:servo_9g xyz="-0.00315 0.0212 0.01105" rpy="${-pi/2} 0 0"/>    <!-- tilt servo (CH3) -->
   </link>
   <joint name="head_tilt_joint" type="revolute">
     <parent link="head_pan_link"/>
     <child  link="head_tilt_link"/>
-    <!-- tilt servo shaft axis, at its top face (where the camera arm sits on the horn) -->
-    <origin xyz="-0.00315 0.0172 0.01105" rpy="0 0 0"/>
+    <!-- tilt servo shaft axis, at its horn face (where the camera arm sits on the horn) -->
+    <origin xyz="-0.00315 0.0212 0.01105" rpy="0 0 0"/>
     <axis xyz="0 1 0"/>
     <!-- safe range CH3: 50..140 deg => -40..+50 deg around home -->
@@ -218,5 +221,5 @@
       </visual>
       <!-- elbow servo (CH4/CH8) in the elbow holder's pocket; its shaft is the bicep axis -->
-      <xacro:servo_9g xyz="0.00045 ${-0.0138*reflect} -0.13455" rpy="${pi/2} ${pi/2} ${(1-reflect)/2*pi}"/>
+      <xacro:servo_9g xyz="0.00045 ${-0.0178*reflect} -0.13455" rpy="${pi/2} ${pi/2} ${(1-reflect)/2*pi}"/>
       </xacro:if>
     </link>
